File: Labs.kicad_pcb (KiCad board)
At the start: 2 copper layers, 85.2 x 61.3 mm, 62 parts, among them J1 PROG_port, J2 USB_C_Receptacle_PowerOnly_6P, Q1 AO3401A, SW1BOOT1 SW_Push, SW2NRST1 SW_Push, U1 STM32F407VGTx, U2 TP4056-42-ESOP8, U3 DW01A, U4 8205A, U5 AMS1117-3.3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

Commit message: fix: minor fixes
Parts:
- C14: moved to F.Cu
- moved C14 33.0 mm to (166.6, 81.6), turned to -90 degrees
Routing:
- net +3.3V: track 183.8 -> 180.3 mm
Changed lines of the file:
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@@
 		)
 	)
+	(footprint "Capacitor_SMD:C_0805_2012Metric_Pad1.18x1.45mm_HandSolder"
+		(layer "F.Cu")
+		(at 166.6 81.6 -90)
+		(descr "Capacitor SMD 0805 (2012 Metric), square (rectangular) end terminal, IPC-7351 nominal with elongated pad for handsoldering. (Body size source: IPC-SM-782 page 76, https://www.pcb-3d.com/wordpress/wp-content/uploads/ipc-sm-782a_amendment_1_and_2.pdf, https://docs.google.com/spreadsheets/d/1BsfQQcO9C6DZCsRaXUlFlo91Tg2WpOkGARC1WS5S8t0/edit?usp=sharing), generated with kicad-footprint-generator")
+		(tags "capacitor handsolder")
+		(property "Reference" "C14"
+			(at 0 -1.68 90)
+			(layer "F.SilkS")
+			(effects
+				(font
+					(size 1 1)
+					(thickness 0.15)
+				)
+			)
+		)
+		(property "Value" "C 10 uF"
+			(at 0 1.68 90)
+			(layer "F.Fab")
+			(effects
+				(font
+					(size 1 1)
+					(thickness 0.15)
+				)
+			)
+		)
+		(property "Datasheet" "~"
+			(at 0 0 90)
+			(layer "F.Fab")
+			(hide yes)
+			(effects
+				(font
+					(size 1.27 1.27)
+					(thickness 0.15)
+				)
+			)
+		)
+		(property "Description" "Unpolarized capacitor"
+			(at 0 0 90)
+			(layer "F.Fab")
+			(hide yes)
+			(effects
+				(font
+					(size 1.27 1.27)
+					(thickness 0.15)
+				)
+			)
+		)
+		(attr smd)
+		(fp_line
+			(start -0.261252 0.735)
+			(end 0.261252 0.735)
+			(stroke
+				(width 0.12)
+				(type solid)
+			)
+			(layer "F.SilkS")
+		)
+		(fp_line
+			(start -0.261252 -0.735)
+			(end 0.261252 -0.735)
+			(stroke
+				(width 0.12)
+				(type solid)
+			)
+			(layer "F.SilkS")
+		)
+		(fp_rect
+			(start -1.88 -0.98)
+			(end 1.88 0.98)
+			(stroke
+				(width 0.05)
+				(type solid)
+			)
+			(fill no)
+			(layer "F.CrtYd")
+		)
+		(fp_rect
+			(start -1 -0.625)
+			(end 1 0.625)
+			(stroke
+				(width 0.1)
+				(type solid)
+			)
+			(fill no)
+			(layer "F.Fab")
+		)
+		(fp_text user "${REFERENCE}"
+			(at 0 0 90)
+			(layer "F.Fab")
+			(effects
+				(font
+					(size 0.5 0.5)
+					(thickness 0.08)
+				)
+			)
+		)
+		(pad "1" smd roundrect
+			(at -1.0375 0 270)
+			(size 1.175 1.45)
+			(layers "F.Cu" "F.Mask" "F.Paste")
+			(roundrect_rratio 0.212766)
+			(net 1 "GND")
+			(pintype "passive")
+		)
+		(pad "2" smd roundrect
+			(at 1.0375 0 270)
+			(size 1.175 1.45)
+			(layers "F.Cu" "F.Mask" "F.Paste")
+			(roundrect_rratio 0.212766)
+			(net 24 "+3.3V")
+			(pintype "passive")
+		)
+		(embedded_fonts no)
+		(model "${KICAD9_3DMODEL_DIR}/Capacitor_SMD.3dshapes/C_0805_2012Metric.step"
+			(offset
+				(xyz 0 0 0)
+			)
+			(scale
+				(xyz 1 1 1)
+			)
+			(rotate
+				(xyz 0 0 0)
+			)
+		)
+	)
 	(footprint "Resistor_SMD:R_0805_2012Metric_Pad1.20x1.40mm_HandSolder"
 		(layer "F.Cu")
@@
 	(footprint "Capacitor_SMD:C_0805_2012Metric_Pad1.18x1.45mm_HandSolder"
 		(layer "B.Cu")
-		(at 134.5575 89.4355)
-		(descr "Capacitor SMD 0805 (2012 Metric), square (rectangular) end terminal, IPC-7351 nominal with elongated pad for handsoldering. (Body size source: IPC-SM-782 page 76, https://www.pcb-3d.com/wordpress/wp-content/uploads/ipc-sm-782a_amendment_1_and_2.pdf, https://docs.google.com/spreadsheets/d/1BsfQQcO9C6DZCsRaXUlFlo91Tg2WpOkGARC1WS5S8t0/edit?usp=sharing), generated with kicad-footprint-generator")
-		(tags "capacitor handsolder")
-		(property "Reference" "C14"
-			(at 0 1.68 0)
-			(layer "B.SilkS")
-			(effects
-				(font
-					(size 1 1)
-					(thickness 0.15)
-				)
-				(justify mirror)
-			)
-		)
-		(property "Value" "C 10 uF"
-			(at 0 -1.68 0)
-			(layer "B.Fab")
-			(effects
-				(font
-					(size 1 1)
-					(thickness 0.15)
-				)
-				(justify mirror)
-			)
-		)
-		(property "Datasheet" "~"
-			(at 0 0 0)
-			(layer "B.Fab")
-			(hide yes)
-			(effects
-				(font
-					(size 1.27 1.27)
-					(thickness 0.15)
-				)
-				(justify mirror)
-			)
-		)
-		(property "Description" "Unpolarized capacitor"
-			(at 0 0 0)
-			(layer "B.Fab")
-			(hide yes)
-			(effects
-				(font
-					(size 1.27 1.27)
-					(thickness 0.15)
-				)
-				(justify mirror)
-			)
-		)
-		(attr smd)
-		(fp_line
-			(start -0.261252 -0.735)
-			(end 0.261252 -0.735)
-			(stroke
-				(width 0.12)
-				(type solid)
-			)
-			(layer "B.SilkS")
-		)
-		(fp_line
-			(start -0.261252 0.735)
-			(end 0.261252 0.735)
-			(stroke
-				(width 0.12)
-				(type solid)
-			)
-			(layer "B.SilkS")
-		)
-		(fp_rect
-			(start -1.88 0.98)
-			(end 1.88 -0.98)
-			(stroke
-				(width 0.05)
-				(type solid)
-			)
-			(fill no)
-			(layer "B.CrtYd")
-		)
-		(fp_rect
-			(start -1 0.625)
-			(end 1 -0.625)
-			(stroke
-				(width 0.1)
-				(type solid)
-			)
-			(fill no)
-			(layer "B.Fab")
-		)
-		(fp_text user "${REFERENCE}"
-			(at 0 0 0)
-			(layer "B.Fab")
-			(effects
-				(font
-					(size 0.5 0.5)
-					(thickness 0.08)
-				)
-				(justify mirror)
-			)
-		)
-		(pad "1" smd roundrect
-			(at -1.0375 0)
-			(size 1.175 1.45)
-			(layers "B.Cu" "B.Mask" "B.Paste")
-			(roundrect_rratio 0.212766)
-			(net 1 "GND")
-			(pintype "passive")
-		)
-		(pad "2" smd roundrect
-			(at 1.0375 0)
-			(size 1.175 1.45)
-			(layers "B.Cu" "B.Mask" "B.Paste")
-			(roundrect_rratio 0.212766)
-			(net 24 "+3.3V")
-			(pintype "passive")
-		)
-		(embedded_fonts no)
-		(model "${KICAD9_3DMODEL_DIR}/Capacitor_SMD.3dshapes/C_0805_2012Metric.step"
-			(offset
-				(xyz 0 0 0)
-			)
-			(scale
-				(xyz 1 1 1)
-			)
-			(rotate
-				(xyz 0 0 0)
-			)
-		)
-	)
-	(footprint "Capacitor_SMD:C_0805_2012Metric_Pad1.18x1.45mm_HandSolder"
-		(layer "B.Cu")
 		(at 116.3575 103.12875 180)
 		(descr "Capacitor SMD 0805 (2012 Metric), square (rectangular) end terminal, IPC-7351 nominal with elongated pad for handsoldering. (Body size source: IPC-SM-782 page 76, https://www.pcb-3d.com/wordpress/wp-content/uploads/ipc-sm-782a_amendment_1_and_2.pdf, https://docs.google.com/spreadsheets/d/1BsfQQcO9C6DZCsRaXUlFlo91Tg2WpOkGARC1WS5S8t0/edit?usp=sharing), generated with kicad-footprint-generator")
@@
 		(layer "Edge.Cuts")
 	)
+	(dimension
+		(type orthogonal)
+		(layer "F.Cu")
+		(pts
+			(xy 109.9075 132.62875) (xy 195.1575 132.62875)
+		)
+		(height 3.52125)
+		(orientation 0)
+		(format
+			(prefix "")
+			(suffix "")
+			(units 3)
+			(units_format 0)
+			(precision 4)
+			(suppress_zeroes yes)
+		)
+		(style
+			(thickness 0.2)
+			(arrow_length 1.27)
+			(text_position_mode 0)
+			(arrow_direction outward)
+			(extension_height 0.58642)
+			(extension_offset 0.5)
+			(keep_text_aligned yes)
+		)
+		(gr_text "85,25"
+			(at 152.5325 134.35 0)
+			(layer "F.Cu")
+			(effects
+				(font
+					(size 1.5 1.5)
+					(thickness 0.3)
+				)
+			)
+		)
+	)
+	(dimension
+		(type orthogonal)
+		(layer "F.Cu")
+		(pts
+			(xy 195.1575 132.62875) (xy 195.1575 71.32875)
+		)
+		(height 3.2425)
+		(orientation 1)
+		(format
+			(prefix "")
+			(suffix "")
+			(units 3)
+			(units_format 0)
+			(precision 4)
+			(suppress_zeroes yes)
+		)
+		(style
+			(thickness 0.2)
+			(arrow_length 1.27)
+			(text_position_mode 0)
+			(arrow_direction outward)
+			(extension_height 0.58642)
+			(extension_offset 0.5)
+			(keep_text_aligned yes)
+		)
+		(gr_text "61,3"
+			(at 196.6 101.97875 90)
+			(layer "F.Cu")
+			(effects
+				(font
+					(size 1.5 1.5)
+					(thickness 0.3)
+				)
+			)
+		)
+	)
 	(segment
 		(start 126.9325 98.05375)
@@
 	)
 	(segment
+		(start 175.0375 75.52875)
+		(end 167.92875 82.6375)
+		(width 0.508)
+		(layer "F.Cu")
+		(net 24)
+	)
+	(segment
 		(start 157.1575 82.67875)
 		(end 163.4575 82.67875)
@@
 	)
 	(segment
-		(start 175.0375 75.52875)
-		(end 167.8875 82.67875)
+		(start 166.55875 82.67875)
+		(end 166.6 82.6375)
 		(width 0.508)
 		(layer "F.Cu")
@@
 	)
 	(segment
-		(start 167.8875 82.67875)
-		(end 163.4575 82.67875)
-		(width 0.508)
-		(layer "F.Cu")
-		(net 24)
-	)
-	(segment
 		(start 124.7575 91.62875)
 		(end 126.1075 91.62875)
@@
 	)
 	(segment
+		(start 167.92875 82.6375)
+		(end 166.6 82.6375)
+		(width 0.508)
+		(layer "F.Cu")
+		(net 24)
+	)
+	(segment
+		(start 163.4575 82.67875)
+		(end 166.55875 82.67875)
+		(width 0.508)
+		(layer "F.Cu")
+		(net 24)
+	)
+	(segment
 		(start 149.4425 92.87375)
 		(end 148.0275 94.28875)
@@
 	)
 	(segment
+		(start 138.1075 85.95)
+		(end 138.1075 83.772252)
+		(width 0.508)
+		(layer "B.Cu")
+		(net 24)
+	)
+	(segment
 		(start 129.1075 94.62875)
 		(end 129.1075 97.87875)
@@
 	)
 	(segment
+		(start 138.072 85.9855)
+		(end 138.1075 85.95)
+		(width 0.508)
+		(layer "B.Cu")
+		(net 24)
+	)
+	(segment
 		(start 129.12 89.4355)
 		(end 129.12 87.67875)
@@
 	)
 	(segment
-		(start 135.595 89.4355)
-		(end 138.10075 89.4355)
-		(width 0.508)
-		(layer "B.Cu")
-		(net 24)
-	)
-	(segment
 		(start 129.12 87.67875)
 		(end 129.12 85.9855)
@@
 	)
 	(segment
-		(start 135.595 89.4355)
-		(end 135.595 85.9855)
-		(width 0.508)
-		(layer "B.Cu")
-		(net 24)
-	)
-	(segment
 		(start 125.1075 80.12875)
 		(end 125.1075 81.12875)
@@
 	(segment
 		(start 138.1075 89.42875)
-		(end 138.1075 83.772252)
+		(end 138.1075 85.95)
 		(width 0.508)
 		(layer "B.Cu")
@@
 	)
 	(segment
-		(start 129.12 82.5355)
-		(end 127.96325 81.37875)
+		(start 135.595 85.9855)
+		(end 138.072 85.9855)
 		(width 0.508)
 		(layer "B.Cu")
@@
 	)
 	(segment
-		(start 138.10075 89.4355)
-		(end 138.1075 89.42875)
+		(start 129.12 82.5355)
+		(end 127.96325 81.37875)
 		(width 0.508)
 		(layer "B.Cu")
